File: zx81c/zx81.kicad_sch (KiCad schematic)
At the start: 72 parts, among them IC1 ZX81ULA, IC2 27C512, IC2B0 ZXROM-SMALL, IC3 Z80CPU, IC4 62256, IC4A0 2114, IC4B0 2114, K1 ZX81CONN, K2 MIC, K3 EAR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

Commit message: updated schematic and pcb to include project credits
Other:
- note added: "Kicad import of Bluescreen2001's Rev C ZX81. Credit to Bluescreen2001 as the origional creator of the project. This conversion was done to allow better maintainability of this brilliant project."
- title: (none) -> Bluescreen2001's ZX81 converted to Kicad
Changed lines of the file:
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@@
 	(generator_version "9.0")
 	(paper "User" 425.45 298.602)
+	(title_block
+		(title "Bluescreen2001's ZX81 converted to Kicad")
+		(date "2025-08-30")
+		(rev "C")
+	)
 	(text "R18"
 		(exclude_from_sim no)
@@
 		)
 	)
+	(text "Kicad import of Bluescreen2001's Rev C ZX81.\nCredit to Bluescreen2001 as the origional creator of the project.\nThis conversion was done to allow better maintainability of this\nbrilliant project."
+		(exclude_from_sim no)
+		(at 308.102 262.382 0)
+		(effects
+			(font
+				(size 1.27 1.27)
+			)
+			(justify left)
+		)
+	)
 	(text "R20"
 		(exclude_from_sim no)
@@
 					(unit 1)
 				)
-			)
-		)
-	)
-	(symbol
-		(lib_id "zx81-c-eagle-import:DINA3_DOC")
-		(at 17.78 279.4 0)
-		(unit 1)
-		(exclude_from_sim no)
-		(in_bom yes)
-		(on_board yes)
-		(dnp no)
-		(property "Reference" "#U$7"
-			(at 17.78 279.4 0)
-			(effects
-				(font
-					(size 1.27 1.27)
-				)
-				(hide yes)
-			)
-		)
-		(property "Value" "DINA3_DOC"
-			(at 17.78 279.4 0)
-			(effects
-				(font
-					(size 1.27 1.27)
-				)
-				(hide yes)
-			)
-		)
-		(property "Footprint" ""
-			(at 17.78 279.4 0)
-			(effects
-				(font
-					(size 1.27 1.27)
-				)
-				(hide yes)
-			)
-		)
-		(property "Datasheet" ""
-			(at 17.78 279.4 0)
-			(effects
-				(font
-					(size 1.27 1.27)
-				)
-				(hide yes)
-			)
-		)
-		(property "Description" ""
-			(at 17.78 279.4 0)
-			(effects
-				(font
-					(size 1.27 1.27)
-				)
-				(hide yes)
-			)
-		)
-		(instances
-			(project ""
-				(path "/eda84689-7afb-43dc-b6dc-7a98674aa9a5"
-					(reference "#U$7")
-					(unit 1)
-				)
